Commit message: completed porting to ros2 humble

File: ur10e_robotiq_description/urdf/ur10e_robotiq.urdf.xacro (robot description, xacro)
@@ -1,9 +1,13 @@
 <?xml version="1.0"?>
 <robot xmlns:xacro="http://ros.org/wiki/xacro" name="ur10e_robotiq" >
+  <xacro:arg name="ur_type" default="ur10e"/>
   <xacro:macro name="ur10e_robotiq" params=
-   "prefix:=''
-    joint_limits_parameters_file:='$(find ur_description)/config/ur10e/joint_limits.yaml'
-    kinematics_parameters_file:='$(find ur_description)/config/ur10e/default_kinematics.yaml'
-    physical_parameters_file:='$(find ur_description)/config/ur10e/physical_parameters.yaml'
+   "name:='ur10e'
+    tf_prefix:='ur10e_'
+    parent:='world'
+    joint_limits_parameters_file:='$(find ur_description)/config/$(arg ur_type)/joint_limits.yaml'
+    kinematics_parameters_file:='$(find ur_description)/config/$(arg ur_type)/default_kinematics.yaml'
+    physical_parameters_file:='$(find ur_description)/config/$(arg ur_type)/physical_parameters.yaml'
+    visual_parameters_file:='$(find ur_description)/config/$(arg ur_type)/visual_parameters.yaml'
     transmission_hw_interface:=hardware_interface/PositionJointInterface
     safety_limits:=false
@@ -11,20 +15,30 @@
     safety_k_position:=20 ">
   <!-- ur10e -->
-  <xacro:include filename="$(find ur_description)/urdf/inc/ur10e_macro.xacro"/>
-  <xacro:ur10e_robot
-    prefix = "${prefix}"
+  <xacro:include filename="$(find ur_description)/urdf/ur_macro.xacro"/>
+  <xacro:ur_robot
+    name="${name}"
+    tf_prefix="${tf_prefix}"
+    parent="${parent}"
     joint_limits_parameters_file="${joint_limits_parameters_file}"
     kinematics_parameters_file="${kinematics_parameters_file}"
     physical_parameters_file="${physical_parameters_file}"
-    visual_parameters_file='$(find ur_description)/config/ur10e/visual_parameters.yaml'
+    visual_parameters_file="${visual_parameters_file}"
     transmission_hw_interface="${transmission_hw_interface}"
     safety_limits="${safety_limits}"
     safety_pos_margin="${safety_pos_margin}"
     safety_k_position="${safety_k_position}"
-  />
+    initial_positions="${dict(shoulder_pan_joint=1.570796327,
+                              shoulder_lift_joint=-2.443460953,
+                              elbow_joint=2.443460953,
+                              wrist_1_joint=-1.570796327,
+                              wrist_2_joint=1.570796327,
+                              wrist_3_joint=0.0,
+                              finger_joint=-0.04)}">
+    <origin xyz="0.0 0.0 0.0" rpy="0.0 0.0 0.0" />
+  </xacro:ur_robot>
   <!-- gripper -->
-  <xacro:include filename="$(find robotiq_2f_85_gripper_visualization)/urdf/robotiq_arg2f_85_model_macro.xacro" />
+  <xacro:include filename="$(find robotiq_description)/urdf/robotiq_2f_85_macro.urdf.xacro" />
   <joint name="rq_coupler_joint" type="fixed">
-    <parent link="tool0" />
+    <parent link="ur10e_tool0" />
     <child  link = "robotiq_coupler" />
     <origin xyz="0 0 0.01" rpy="0 0 ${0.5*pi}" />
@@ -56,8 +70,10 @@
   <joint name="robotiq_joint" type="fixed">
     <parent link="robotiq_coupler" />
-    <child link = "robotiq_arg2f_base_link" />
+    <child link = "robotiq_85_base_link" />
     <origin xyz="0.0 0.0 0.0" rpy="0 0 ${0.0*pi}" />
   </joint>
-    <xacro:robotiq_arg2f_85 prefix=""/>
+  <xacro:robotiq_gripper prefix="" name="robotiq_2f_85" parent="robotiq_coupler">
+    <origin xyz="0 0 0.0" rpy="0 0 0" />
+  </xacro:robotiq_gripper>
   <link name="open_tip" />
   <joint name="open_tip_joint" type="fixed">

File: ur10e_robotiq_description/urdf/ur10e_robotiq_robot.urdf.xacro (robot description, xacro)
@@ -4,3 +4,4 @@
   <xacro:include filename="$(find ur10e_robotiq_description)/urdf/ur10e_robotiq.urdf.xacro" />
   <xacro:ur10e_robotiq /> <!--DO NOT DELETE -->
+  <link name="world" />
 </robot>
