Commit message: created moveit_config and bringup packages

File: ur_robotiq_description/urdf/ur_robotiq.urdf.xacro (robot description, xacro)
@@ -12,4 +12,9 @@
   <xacro:arg name="tool_tcp_port" default="54321"/>
   <xacro:arg name="headless_mode" default="false"/>
+  <xacro:arg name="robotiq_use_socket_communication" default="false"/>
+  <xacro:arg name="robotiq_ip_address" default="192.168.10.2" />
+  <xacro:arg name="robotiq_port" default="63352" />
+  <xacro:arg name="robotiq_connection_timeout" default="30000" /> <!-- milliseconds -->
+  <xacro:arg name="robotiq_activate_gripper_by_default" default="1" /> <!-- 0: false, 1: true -->
   <!-- UR properties -->
   <xacro:property name="joint_limit_params" value="$(find ur_robotiq_description)/config/$(arg ur_type)/joint_limits.yaml"/>
@@ -99,4 +104,9 @@
     robotiq_mock_sensor_commands="${robotiq_mock_sensor_commands}"
     robotiq_include_ros2_control="${robotiq_include_ros2_control}"
+    robotiq_use_socket_communication="$(arg robotiq_use_socket_communication)"
+    robotiq_ip_address="$(arg robotiq_ip_address)"
+    robotiq_port="$(arg robotiq_port)"
+    robotiq_connection_timeout="$(arg robotiq_connection_timeout)"
+    robotiq_activate_gripper_by_default="$(arg robotiq_activate_gripper_by_default)"
   />
 </robot>

File: ur_robotiq_description/urdf/ur_robotiq.xacro (robot description, xacro)
@@ -62,5 +62,10 @@
     robotiq_isaac_joint_states:=/isaac_joint_states
     robotiq_mock_sensor_commands:=false
-    robotiq_include_ros2_control:=true">
+    robotiq_include_ros2_control:=true
+    robotiq_use_socket_communication:=false
+    robotiq_ip_address:=192.168.10.2
+    robotiq_port:=63352
+    robotiq_connection_timeout:=30000
+    robotiq_activate_gripper_by_default:=1">
   <!-- UR robot -->
   <xacro:include filename="$(find ur_description)/urdf/ur_macro.xacro"/>
@@ -152,5 +157,10 @@
     mock_sensor_commands="${robotiq_mock_sensor_commands}"
     include_ros2_control="${robotiq_include_ros2_control}"
-    com_port="${tool_device_name}">
+    com_port="${tool_device_name}"
+    use_socket_communication="${robotiq_use_socket_communication}"
+    ip_address="${robotiq_ip_address}"
+    port="${robotiq_port}"
+    connection_timeout="${robotiq_connection_timeout}"
+    activate_gripper_by_default="${robotiq_activate_gripper_by_default}">
     <origin xyz="0 0 0" rpy="0 0 ${-0.5*pi}" />
   </xacro:robotiq_gripper>

File: ur_robotiq_moveit_config/config/ur_robotiq.ros2_control.xacro (robot description, xacro)
@@ -50,11 +50,4 @@
                 <state_interface name="velocity"/>
             </joint>
-            <joint name="robotiq_85_left_knuckle_joint">
-                <command_interface name="position"/>
-                <state_interface name="position">
-                  <param name="initial_value">${initial_positions['robotiq_85_left_knuckle_joint']}</param>
-                </state_interface>
-                <state_interface name="velocity"/>
-            </joint>
         </ros2_control>
     </xacro:macro>
